Commit message: save

File: pendulum/urdf/pendulum.ros2_control.xacro (robot description, xacro)
@@ -2,11 +2,15 @@
 <robot xmlns:xacro="http://www.ros.org/wiki/xacro">
     <xacro:macro name="pendulum_ros2_control">
-        <ros2_control name="SingleJointSystem" type="system">
+        <ros2_control name="pendulumeSystem" type="system">
             <hardware>
                 <plugin>gazebo_ros2_control/GazeboSystem</plugin>
             </hardware>
             <joint name="cart_to_pole1">
-                <command_interface name="position" />
-                <command_interface name="velocity" />
+                <command_interface name="effort" />
+                <state_interface name="position" />
+                <state_interface name="velocity" />
+                <state_interface name="effort" />
+            </joint>
+            <joint name="base_to_plat">
                 <command_interface name="effort" />
                 <state_interface name="position" />
@@ -19,7 +23,4 @@
                 <parameters>$(find pendulum)/config/pendulum_ros2_controller.yaml</parameters>
             </plugin>
-            <ros>
-                <remapping>/pendulum/joint_states:=/joint_states</remapping>
-            </ros>
         </gazebo>
     </xacro:macro>

Commit message: 循环跑通

File: pendulum/urdf/pendulum.ros2_control.xacro (robot description, xacro)
@@ -6,5 +6,5 @@
                 <plugin>gazebo_ros2_control/GazeboSystem</plugin>
             </hardware>
-            <joint name="cart_to_pole1">
+            <joint name="base_to_plat">
                 <command_interface name="effort" />
                 <state_interface name="position" />
@@ -12,5 +12,5 @@
                 <state_interface name="effort" />
             </joint>
-            <joint name="base_to_plat">
+            <joint name="cart_to_pole1">
                 <command_interface name="effort" />
                 <state_interface name="position" />
