Commit message: 简化代码

File: pendulum/urdf/cartpole_body.urdf.xacro (robot description, xacro)
@@ -47,14 +47,4 @@
             <dynamics damping="0.0" friction="0.0" />
         </joint>
-        <transmission name="tran2">
-            <type>transmission_interface/SimpleTransmission</type>
-            <joint name="base_to_plat">
-                <hardwareInterface>hardware_interface/EffortJointInterface</hardwareInterface>
-            </joint>
-            <actuator name="planar_motor_2">
-                <hardwareInterface>hardware_interface/EffortJointInterface</hardwareInterface>
-                <mechanicalReduction>1</mechanicalReduction>
-            </actuator>
-        </transmission>
         <link name="pole1">
             <visual>
@@ -81,14 +71,4 @@
             <limit effort="100000.0" lower="-3.14" upper="3.14" velocity="50" />
         </joint>
-        <transmission name="tran3">
-            <type>transmission_interface/SimpleTransmission</type>
-            <joint name="cart_to_pole1">
-                <hardwareInterface>hardware_interface/EffortJointInterface</hardwareInterface>
-            </joint>
-            <actuator name="rev_motor">
-                <hardwareInterface>hardware_interface/EffortJointInterface</hardwareInterface>
-                <mechanicalReduction>1</mechanicalReduction>
-            </actuator>
-        </transmission>
     </xacro:macro>
 </robot>

Commit message: save

File: pendulum/urdf/cartpole_body.urdf.xacro (robot description, xacro)
@@ -7,5 +7,5 @@
             <visual>
                 <geometry>
-                    <box size="30 0.05 0.05" />
+                    <box size="300 0.05 0.05" />
                 </geometry>
                 <origin xyz="0 0 0" />
@@ -47,14 +47,4 @@
             <dynamics damping="0.0" friction="0.0" />
         </joint>
-        <transmission name="tran2">
-            <type>transmission_interface/SimpleTransmission</type>
-            <joint name="base_to_plat">
-                <hardwareInterface>hardware_interface/EffortJointInterface</hardwareInterface>
-            </joint>
-            <actuator name="planar_motor_2">
-                <hardwareInterface>hardware_interface/EffortJointInterface</hardwareInterface>
-                <mechanicalReduction>1</mechanicalReduction>
-            </actuator>
-        </transmission>
         <link name="pole1">
             <visual>
@@ -74,5 +64,5 @@
         </gazebo>
         <joint name="cart_to_pole1" type="revolute">
-            <axis xyz="0 1 0" />
+            <axis xyz="0 0 0" />
             <origin xyz="0.0 0.0 0" rpy="0.0 0.0 0.0" />
             <parent link="cart" />
@@ -81,14 +71,4 @@
             <limit effort="100000.0" lower="-3.14" upper="3.14" velocity="50" />
         </joint>
-        <!-- <transmission name="tran3">
-            <type>transmission_interface/SimpleTransmission</type>
-            <joint name="cart_to_pole1">
-                <hardwareInterface>hardware_interface/EffortJointInterface</hardwareInterface>
-            </joint>
-            <actuator name="rev_motor">
-                <hardwareInterface>hardware_interface/EffortJointInterface</hardwareInterface>
-                <mechanicalReduction>1</mechanicalReduction>
-            </actuator>
-        </transmission> -->
     </xacro:macro>
 </robot>

Commit message: save

File: pendulum/urdf/cartpole_body.urdf.xacro (robot description, xacro)
@@ -44,5 +44,5 @@
             <parent link="slideBar" />
             <child link="cart" />
-            <limit effort="100000.0" lower="-15" upper="15" velocity="100" />
+            <limit effort="100000.0" lower="-150" upper="150" velocity="100" />
             <dynamics damping="0.0" friction="0.0" />
         </joint>
@@ -64,5 +64,5 @@
         </gazebo>
         <joint name="cart_to_pole1" type="revolute">
-            <axis xyz="0 0 0" />
+            <axis xyz="0 1 0" />
             <origin xyz="0.0 0.0 0" rpy="0.0 0.0 0.0" />
             <parent link="cart" />
